Commit message: update car.urdf

File: testpkg0/urdf/lab9/car.urdf (robot description, URDF)
Before this commit: robot car0, 6 links, 5 joints
Joints:
- joint base_to_left_wheel0: type continuous -> fixed
- joint base_to_left_wheel1: type continuous -> fixed
- joint base_to_right_wheel0: type continuous -> fixed
- joint base_to_right_wheel1: type continuous -> fixed
